File: LCD_Disp_AIR_NTCand Connector.sch (EAGLE design)
At the start: 14 parts, among them Q1 2N2219

Commit message: added fuel pressure and oil pressure from solid state sensors -- updated interconnect diagram
Connections:
- net N$3: now also X1.9
Other:
- note added: "FP 5V , pin 9, FP-Gnd 1"
Changed lines of the file:
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@@
 <text x="181.864" y="186.182" size="1.778" layer="97">2nd in NTC</text>
 <text x="111.76" y="193.04" size="1.778" layer="97">2nd NTC out</text>
+<text x="228.6" y="223.52" size="1.778" layer="95">FP 5V , pin 9, FP-Gnd 1 </text>
 </plain>
 <instances>
@@
 <wire x1="149.86" y1="210.82" x2="160.02" y2="210.82" width="0.1524" layer="91"/>
 <junction x="160.02" y="210.82"/>
+<pinref part="X1" gate="-1" pin="9"/>
+<wire x1="116.84" y1="231.14" x2="116.84" y2="243.84" width="0.1524" layer="91"/>
+<wire x1="116.84" y1="243.84" x2="177.8" y2="243.84" width="0.1524" layer="91"/>
+<wire x1="177.8" y1="243.84" x2="177.8" y2="210.82" width="0.1524" layer="91"/>
+<wire x1="177.8" y1="210.82" x2="170.18" y2="210.82" width="0.1524" layer="91"/>
 </segment>
 </net>
